Commit message: mvp setup

File: float_description/urdf/base_v1-1.urdf.xacro (robot description, xacro)
@@ -5,5 +5,5 @@
             <origin xyz="0.0 0.0 0.0" rpy="0.0 0.0 0.0"/>
             <geometry>
-                <mesh filename="package://alpha_description/mesh/float_assembly.stl" scale="0.001 0.001 0.001"/>
+                <mesh filename="package://float_description/mesh/float_assembly.stl" scale="0.001 0.001 0.001"/>
             </geometry>
         </visual>
@@ -15,7 +15,7 @@
         <child link="cg_link"/>
     </joint>
-    <!-- <link name="imu"/>
+    <link name="imu"/>
     <joint name="imu_joint" type="fixed">
-        <origin xyz="-0.0465 0.060 0.14648" rpy="3.14159265359 0.0 0.0"/>
+        <origin xyz="-0.0465 0.060 0.14648" rpy="0.0 0.0 0.0"/>
         <parent link="base_link"/>
         <child link="imu"/>
@@ -23,5 +23,5 @@
     <link name="gps"/>
     <joint name="gps_joint" type="fixed">
-        <origin xyz="0.1 0.0 0.407241" rpy="3.1415 0.0 0.0"/>
+        <origin xyz="-0.2 0.0 0.0" rpy="0.0 0.0 0.0"/>
         <parent link="base_link"/>
         <child link="gps"/>
@@ -29,5 +29,5 @@
     <link name="pressure"/>
     <joint name="pressure_joint" type="fixed">
-        <origin xyz="-0.187845 -0.060 0.124465" rpy="0.0 3.14159265359 0.0"/>
+        <origin xyz="0.2 0.0 0.0" rpy="0.0 0.0 0.0"/>
         <parent link="base_link"/>
         <child link="pressure"/>
@@ -35,5 +35,5 @@
     <link name="heave_port_thruster_link"/>
     <joint name="heave_port_thruster_joint" type="fixed">
-        <origin xyz="-0.554 0.0 0.100" rpy="0.0 0.0 0.0"/>
+        <origin xyz="0.2 0.11 0.0" rpy="0.0 1.57 0.0"/>
         <parent link="base_link"/>
         <child link="heave_port_thruster_link"/>
@@ -41,7 +41,7 @@
     <link name="heave_stbd_thruster_link"/>
     <joint name="heave_stbd_thruster_joint" type="fixed">
-        <origin xyz="0.48735 0.0 0.089" rpy="0.0 1.57079632679 0.0"/>
+        <origin xyz="0.2 -0.11 0.0" rpy="0.0 1.57 0.0"/>
         <parent link="base_link"/>
         <child link="heave_stbd_thruster_link"/>
-    </joint> -->
+    </joint>
 </robot>

Commit message: make rviz and sf consistent on thruster

File: float_description/urdf/base_v1-1.urdf.xacro (robot description, xacro)
@@ -35,5 +35,5 @@
     <link name="heave_port_thruster_link"/>
     <joint name="heave_port_thruster_joint" type="fixed">
-        <origin xyz="0.2 0.11 0.0" rpy="0.0 1.57 0.0"/>
+        <origin xyz="0.2 0.11 0.0" rpy="0.0 -1.57 0.0"/>
         <parent link="base_link"/>
         <child link="heave_port_thruster_link"/>
@@ -41,5 +41,5 @@
     <link name="heave_stbd_thruster_link"/>
     <joint name="heave_stbd_thruster_joint" type="fixed">
-        <origin xyz="0.2 -0.11 0.0" rpy="0.0 1.57 0.0"/>
+        <origin xyz="0.2 -0.11 0.0" rpy="0.0 -1.57 0.0"/>
         <parent link="base_link"/>
         <child link="heave_stbd_thruster_link"/>

Commit message: urdf configured, rviz checked, goto_depth controller works

File: float_description/urdf/base_v1-1.urdf.xacro (robot description, xacro)
@@ -11,15 +11,15 @@
     <link name="cg_link"/>
     <joint name="cg_joint" type="fixed">
-        <origin xyz="0.100 0.000 0.10" rpy="3.14159265359 0.0 0.0"/>
+        <origin xyz="0.0 0.000 0.0" rpy="0.0 0.0 0.0"/>
         <parent link="base_link"/>
         <child link="cg_link"/>
     </joint>
-    <link name="imu"/>
+    <!-- <link name="imu"/>
     <joint name="imu_joint" type="fixed">
         <origin xyz="-0.0465 0.060 0.14648" rpy="0.0 0.0 0.0"/>
         <parent link="base_link"/>
         <child link="imu"/>
-    </joint>
-    <link name="gps"/>
+    </joint> -->
+    <!-- <link name="gps"/>
     <joint name="gps_joint" type="fixed">
         <origin xyz="-0.2 0.0 0.0" rpy="0.0 0.0 0.0"/>
@@ -32,8 +32,8 @@
         <parent link="base_link"/>
         <child link="pressure"/>
-    </joint>
+    </joint> -->
     <link name="heave_port_thruster_link"/>
     <joint name="heave_port_thruster_joint" type="fixed">
-        <origin xyz="0.2 0.11 0.0" rpy="0.0 -1.57 0.0"/>
+        <origin xyz="-0.2 -0.11 0.0" rpy="0.0 0.0 0.0"/>
         <parent link="base_link"/>
         <child link="heave_port_thruster_link"/>
@@ -41,5 +41,5 @@
     <link name="heave_stbd_thruster_link"/>
     <joint name="heave_stbd_thruster_joint" type="fixed">
-        <origin xyz="0.2 -0.11 0.0" rpy="0.0 -1.57 0.0"/>
+        <origin xyz="-0.2 0.11 0.0" rpy="0.0 0.0 0.0"/>
         <parent link="base_link"/>
         <child link="heave_stbd_thruster_link"/>

Commit message: testing movable thruster

File: float_description/urdf/base_v1-1.urdf.xacro (robot description, xacro)
@@ -15,10 +15,10 @@
         <child link="cg_link"/>
     </joint>
-    <!-- <link name="imu"/>
+    <link name="imu"/>
     <joint name="imu_joint" type="fixed">
-        <origin xyz="-0.0465 0.060 0.14648" rpy="0.0 0.0 0.0"/>
+        <origin xyz="-0.2 0.0 0.0" rpy="0.0 1.5707 0.0"/>
         <parent link="base_link"/>
         <child link="imu"/>
-    </joint> -->
+    </joint>
     <!-- <link name="gps"/>
     <joint name="gps_joint" type="fixed">
